Commit message: Fix : sensor foramt & angles

File: descriptions/go1_description/xacro/depthCamera.xacro (robot description, xacro)
@@ -42,5 +42,5 @@
                         <width>928</width>
                         <height>800</height>
-                        <format>R8G8B8</format>
+                        <format>B8G8R8</format>
                     </image>
                     <clip>

File: descriptions/go1_description/xacro/gazebo.xacro (robot description, xacro)
@@ -92,5 +92,5 @@
                     <width>928</width>
                     <height>800</height>
-                    <format>R8G8B8</format>
+                    <format>B8G8R8</format>
                 </image>
                 <depth_camera></depth_camera>
@@ -134,5 +134,5 @@
           <width>640</width>
           <height>480</height>
-          <format>R8G8B8</format>
+          <format>B8G8R8</format>
         </image>
         <clip>

File: descriptions/go1_description/xacro/robot.xacro (robot description, xacro)
@@ -13,4 +13,5 @@
     <xacro:property name="rolloverProtection" value="false"/>
     <!-- Debug mode will hung up the robot, use "true" or "false" to switch it. -->
+    <xacro:arg name="DEBUG" value="false" default="false"/>
     <xacro:if value="$(arg DEBUG)">
         <link name="world"/>
@@ -124,17 +125,17 @@
     </xacro:leg>
     <xacro:depthCamera camID="1" name="face">
-        <origin rpy="${PI} 0 0" xyz="0.2785 0.0125 0.0167"/>
+        <origin rpy="0 0 0" xyz="0.2785 0.0125 0.0167"/>
     </xacro:depthCamera>
     <xacro:depthCamera camID="2" name="chin">
-        <origin rpy="${PI} ${PI/2} 0" xyz="0.2522 0.0125 -0.0436"/>
+        <origin rpy="0 ${PI/2} 0" xyz="0.2522 0.0125 -0.0436"/>
     </xacro:depthCamera>
     <xacro:depthCamera camID="3" name="left">
-        <origin rpy="${PI} 0.2618 ${PI/2}" xyz="-0.066 0.082 -0.0176"/>
+        <origin rpy="0 0.2618 ${PI/2}" xyz="-0.066 0.082 -0.0176"/>
     </xacro:depthCamera>
     <xacro:depthCamera camID="4" name="right">
-        <origin rpy="${PI} 0.2618 ${-PI/2}" xyz="-0.041 -0.082 -0.0176"/>
+        <origin rpy="0 0.2618 ${-PI/2}" xyz="-0.041 -0.082 -0.0176"/>
     </xacro:depthCamera>
     <xacro:depthCamera camID="5" name="rearDown">
-        <origin rpy="${PI} ${PI/2} 0" xyz="-0.0825 0.0125 -0.04365"/>
+        <origin rpy="0 ${PI/2} 0" xyz="-0.0825 0.0125 -0.04365"/>
     </xacro:depthCamera>
     <joint name="camera_laserscan_joint_left" type="fixed">
